File: analogInputtStagev0.3.2/analogInputtStagev0.3.2.kicad_sch (KiCad schematic)
At the start: 17 parts, among them J1 Conn_01x03_Male_Pin, J2 Conn_01x03_Female_Pin, J3 AudioJack2_SwitchT, U1 MCP6004

Commit message: Uploading KiCAD Versions
Parts:
- renumbered D2 to D10, D3 to D11, D4 to D12, D1 to D9, J1 to J7, J2 to J8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
