File: Oblique Palette 0.5.1 PCB/Oblique Palette 0.5.1 PCB Output/Oblique Palette 0.5.1 PCB Output.kicad_sch (KiCad schematic)
At the start: 25 parts

Commit message: PCB 0.5.2
Parts:
- U?: now fitted
Changed lines of the file:
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@@
 		(in_bom yes)
 		(on_board yes)
-		(dnp yes)
+		(dnp no)
 		(fields_autoplaced yes)
 		(property "Reference" "U?"
@@
 		)
 	)
+	(sheet_instances
+		(path "/"
+			(page "1")
+		)
+	)
