File: Oblique Palette 0.5.1 PCB/Oblique Palette 0.5.1 PCB Input/Oblique Palette 0.5.1 PCB Input.kicad_sch (KiCad schematic)
At the start: 18 parts, among them J16 Conn_01x03_Female_Pin, J17 AudioJack2_SwitchT, U3 MCP6004

Commit message: I've cleaned up all sorts of misplaced resistors. Manually routing input channel 1 to replicate across inputs.
Parts:
- R160: value 2K -> 200K
- R68: value 1K -> 100K
Changed lines of the file:
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@@
 			)
 		)
-		(property "Value" "1K"
+		(property "Value" "100K"
 			(at 105.41 83.8199 0)
 			(effects
@@
 			)
 		)
-		(property "Value" "2K"
+		(property "Value" "200K"
 			(at 96.266 83.312 90)
 			(effects
