File: Oblique Palette 0.5.x PCB Files/Oblique Palette 0.5.4 PCB Main/Oblique Palette 0.5.4 PCB Main.kicad_sch (KiCad schematic)
At the start: 18 parts, among them J11 Conn_01x03_Male_Pin, J13 Conn_01x03_Male_Pin, J14 Conn_01x03_Male_Pin, J2 Conn_01x03_Male_Pin, J4 Conn_01x03_Male_Pin, J5 Conn_01x03_Male_Pin, J7 Conn_01x03_Male_Pin, J9 Conn_01x03_Male_Pin, U1 CD4051B, U2 Pico

Commit message: Making traces beautiful.
Changed lines of the file:
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@@
+	)
+	(symbol
+		(lib_id "power:VCC")
+		(at 273.05 31.75 180)
+		(unit 1)
+		(exclude_from_sim no)
+		(in_bom yes)
+		(on_board yes)
+		(dnp no)
+		(fields_autoplaced yes)
+		(property "Reference" "#PWR068"
+			(at 273.05 27.94 0)
+			(effects
+				(font
+					(size 1.27 1.27)
+				)
+				(hide yes)
+			)
+		)
+		(property "Value" "+3.3V"
+			(at 273.05 36.83 0)
+			(effects
+				(font
+					(size 1.27 1.27)
+				)
+			)
+		)
+		(property "Footprint" ""
+			(at 273.05 31.75 0)
+			(effects
+				(font
+					(size 1.27 1.27)
+				)
+				(hide yes)
+			)
+		)
+		(property "Datasheet" ""
+			(at 273.05 31.75 0)
+			(effects
+				(font
+					(size 1.27 1.27)
+				)
+				(hide yes)
+			)
+		)
+		(property "Description" "Power symbol creates a global label with name \"VCC\""
+			(at 273.05 31.75 0)
+			(effects
+				(font
+					(size 1.27 1.27)
+				)
+				(hide yes)
+			)
+		)
+		(pin "1"
+		)
+		(instances
+			(project "Oblique Palette 0.5.4 PCB Main"
+				(path "/28718c51-05fa-44bf-9e59-30883fb9ecef"
+					(reference "#PWR068")
+					(unit 1)
+				)
+			)
+		)
 	)
 	(symbol
@@
 	)
 	(symbol
+		(lib_id "power:PWR_FLAG")
+		(at 273.05 31.75 0)
+		(unit 1)
+		(exclude_from_sim no)
+		(in_bom yes)
+		(on_board yes)
+		(dnp no)
+		(fields_autoplaced yes)
+		(property "Reference" "#FLG03"
+			(at 273.05 29.845 0)
+			(effects
+				(font
+					(size 1.27 1.27)
+				)
+				(hide yes)
+			)
+		)
+		(property "Value" "PWR_FLAG"
+			(at 273.05 27.305 0)
+			(effects
+				(font
+					(size 1.27 1.27)
+				)
+			)
+		)
+		(property "Footprint" ""
+			(at 273.05 31.75 0)
+			(effects
+				(font
+					(size 1.27 1.27)
+				)
+				(hide yes)
+			)
+		)
+		(property "Datasheet" "~"
+			(at 273.05 31.75 0)
+			(effects
+				(font
+					(size 1.27 1.27)
+				)
+				(hide yes)
+			)
+		)
+		(property "Description" "Special symbol for telling ERC where power comes from"
+			(at 273.05 31.75 0)
+			(effects
+				(font
+					(size 1.27 1.27)
+				)
+				(hide yes)
+			)
+		)
+		(pin "1"
+		)
+		(instances
+			(project "Oblique Palette 0.5.4 PCB Main"
+				(path "/28718c51-05fa-44bf-9e59-30883fb9ecef"
+					(reference "#FLG03")
+					(unit 1)
+				)
+			)
+		)
+	)
+	(symbol
 		(lib_id "power:GNDREF")
 		(at 187.96 154.94 0)
@@
 		)
 		(instances
-			(project "Oblique Palette 0.5.1 PCB Main"
+			(project "Oblique Palette 0.5.4 PCB Main"
 				(path "/28718c51-05fa-44bf-9e59-30883fb9ecef"
 					(page "11")
@@
 		)
 		(instances
-			(project "Oblique Palette 0.5.1 PCB Main"
+			(project "Oblique Palette 0.5.4 PCB Main"
 				(path "/28718c51-05fa-44bf-9e59-30883fb9ecef"
 					(page "4")
@@
 		)
 		(instances
-			(project "Oblique Palette 0.5.1 PCB Main"
+			(project "Oblique Palette 0.5.4 PCB Main"
 				(path "/28718c51-05fa-44bf-9e59-30883fb9ecef"
 					(page "15")
@@
 		)
 		(instances
-			(project "Oblique Palette 0.5.1 PCB Main"
+			(project "Oblique Palette 0.5.4 PCB Main"
 				(path "/28718c51-05fa-44bf-9e59-30883fb9ecef"
 					(page "2")
@@
 		)
 		(instances
-			(project "Oblique Palette 0.5.1 PCB Main"
+			(project "Oblique Palette 0.5.4 PCB Main"
 				(path "/28718c51-05fa-44bf-9e59-30883fb9ecef"
 					(page "13")
@@
 		)
 		(instances
-			(project "Oblique Palette 0.5.1 PCB Main"
+			(project "Oblique Palette 0.5.4 PCB Main"
 				(path "/28718c51-05fa-44bf-9e59-30883fb9ecef"
 					(page "12")
@@
 		)
 		(instances
-			(project "Oblique Palette 0.5.1 PCB Main"
+			(project "Oblique Palette 0.5.4 PCB Main"
 				(path "/28718c51-05fa-44bf-9e59-30883fb9ecef"
 					(page "8")
@@
 		)
 		(instances
-			(project "Oblique Palette 0.5.1 PCB Main"
+			(project "Oblique Palette 0.5.4 PCB Main"
 				(path "/28718c51-05fa-44bf-9e59-30883fb9ecef"
 					(page "9")
@@
 		)
 		(instances
-			(project "Oblique Palette 0.5.1 PCB Main"
+			(project "Oblique Palette 0.5.4 PCB Main"
 				(path "/28718c51-05fa-44bf-9e59-30883fb9ecef"
 					(page "7")
@@
 		)
 		(instances
-			(project "Oblique Palette 0.5.1 PCB Main"
+			(project "Oblique Palette 0.5.4 PCB Main"
 				(path "/28718c51-05fa-44bf-9e59-30883fb9ecef"
 					(page "16")
@@
 		)
 		(instances
-			(project "Oblique Palette 0.5.1 PCB Main"
+			(project "Oblique Palette 0.5.4 PCB Main"
 				(path "/28718c51-05fa-44bf-9e59-30883fb9ecef"
 					(page "6")
@@
 		)
 		(instances
-			(project "Oblique Palette 0.5.1 PCB Main"
+			(project "Oblique Palette 0.5.4 PCB Main"
 				(path "/28718c51-05fa-44bf-9e59-30883fb9ecef"
 					(page "3")
@@
 		)
 		(instances
-			(project "Oblique Palette 0.5.1 PCB Main"
+			(project "Oblique Palette 0.5.4 PCB Main"
 				(path "/28718c51-05fa-44bf-9e59-30883fb9ecef"
 					(page "14")
@@
 		)
 		(instances
-			(project "Oblique Palette 0.5.1 PCB Main"
+			(project "Oblique Palette 0.5.4 PCB Main"
 				(path "/28718c51-05fa-44bf-9e59-30883fb9ecef"
 					(page "10")
@@
 		)
 		(instances
-			(project "Oblique Palette 0.5.1 PCB Main"
+			(project "Oblique Palette 0.5.4 PCB Main"
 				(path "/28718c51-05fa-44bf-9e59-30883fb9ecef"
 					(page "1")
@@
 		)
 		(instances
-			(project "Oblique Palette 0.5.1 PCB Main"
+			(project "Oblique Palette 0.5.4 PCB Main"
 				(path "/28718c51-05fa-44bf-9e59-30883fb9ecef"
 					(page "5")
