File: Oblique Palette 0.5.x PCB Files/Oblique Palette 0.5.4 PCB Main/_autosave-Oblique Palette 0.5.4 PCB Main.kicad_sch (KiCad schematic)
At the start: 6 parts, among them U1 CD4051B, U2 Pico

Commit message: Looks like I just about finished up, only to realize that KiCAD re-designated all components.
I think the PCB is all correct now, but it no longer matches the schematic. Committing now so I can roll back and redo with more incremental commits.
Parts:
- renumbered R2 to R1, R9 to R2, R1 to R3, R10 to R4
