File: Oblique Palette 0.5.x PCB Files/Oblique Palette 0.5.4 PCB Main/servoOut.kicad_sch (KiCad schematic)
At the start: 3 parts, among them J3 Conn_01x03_Male_Pin

Commit message: Might be ready for manufacture. Weird warning that says that the power caps are specified with a through-hole footprint, which they aren't.
Parts:
- C18: footprint Capacitor_THT:CP_Radial_D5.0mm_P2.50mm -> Capacitor_SMD:CP_Elec_10x10.5
Changed lines of the file:
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@@
 			)
 		)
-		(property "Footprint" "Capacitor_THT:CP_Radial_D5.0mm_P2.50mm"
+		(property "Footprint" "Capacitor_SMD:CP_Elec_10x10.5"
 			(at 139.7 100.33 0)
 			(effects
