File: Oblique Palette 0.5.x PCB Files/Oblique Palette 0.5.1 PCB Input/Oblique Palette 0.5.1 PCB Input.kicad_sch (KiCad schematic)
At the start: 18 parts, among them J16 Conn_01x03_Female_Pin, J17 AudioJack2_SwitchT, U3 MCP6004

Commit message: Making traces beautiful.
Changed lines of the file:
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@@
 		)
 	)
-	(hierarchical_label "3v3"
+	(hierarchical_label "+3.3V"
 		(shape input)
 		(at 110.49 38.1 270)

Commit message: Might be ready for manufacture. Weird warning that says that the power caps are specified with a through-hole footprint, which they aren't.
Parts:
- U3: LCSC PN (none) -> C116668
Changed lines of the file:
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@@
+			)
+		)
+		(property "LCSC PN" "C116668"
+			(at 173.99 105.41 0)
+			(effects
+				(font
+					(size 1.27 1.27)
+				)
+				(hide yes)
 			)
 		)
@@
 			)
 		)
+		(property "LCSC PN" "C116668"
+			(at 105.41 105.41 0)
+			(effects
+				(font
+					(size 1.27 1.27)
+				)
+				(hide yes)
+			)
+		)
 		(pin "12"
 		)
@@
 			)
 		)
+		(property "LCSC PN" "C116668"
+			(at 152.4 105.41 0)
+			(effects
+				(font
+					(size 1.27 1.27)
+				)
+				(hide yes)
+			)
+		)
 		(pin "12"
 		)
@@
 			)
 		)
+		(property "LCSC PN" "C116668"
+			(at 130.81 105.41 0)
+			(effects
+				(font
+					(size 1.27 1.27)
+				)
+				(hide yes)
+			)
+		)
 		(pin "12"
 		)
@@
 			(at 173.99 105.41 0)
 			(effects
+				(font
+					(size 1.27 1.27)
+				)
+				(hide yes)
+			)
+		)
+		(property "LCSC PN" "C116668"
+			(at 173.99 105.41 0)
+			(effects

Commit message: Ready to go, but for some blank part numbers in the BOM to work out with the manufacturer.
Parts:
- D2, D3, D6: footprint LED_THT:LED_SideEmitter_Rectangular_W4.5mm_H1.6mm -> LED_THT:LED_Rectangular_W5.0mm_H2.0mm; symbol LED:IRL81A -> Device:LED
Changed lines of the file:
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@@
 	)
 	(junction
-		(at 130.81 120.65)
-		(diameter 0)
-		(color 0 0 0 0)
-	)
-	(junction
 		(at 162.56 60.96)
 		(diameter 0)
@@
 	)
 	(junction
+		(at 130.81 120.65)
+		(diameter 0)
+		(color 0 0 0 0)
+	)
+	(junction
 		(at 149.86 78.74)
 		(diameter 0)
@@
 	)
 	(symbol
-		(lib_id "LED:IRL81A")
-		(at 130.81 115.57 90)
+		(lib_id "Device:LED")
+		(at 130.81 116.84 90)
 		(unit 1)
 		(exclude_from_sim no)
@@
 		(fields_autoplaced yes)
 		(property "Reference" "D2"
-			(at 133.35 115.4429 90)
+			(at 134.62 117.1574 90)
 			(effects
 				(font
@@
 		)
 		(property "Value" "White"
-			(at 133.35 117.9829 90)
+			(at 134.62 119.6974 90)
 			(effects
 				(font
@@
 			)
 		)
-		(property "Footprint" "LED_THT:LED_SideEmitter_Rectangular_W4.5mm_H1.6mm"
-			(at 126.365 115.57 0)
+		(property "Footprint" "LED_THT:LED_Rectangular_W5.0mm_H2.0mm"
+			(at 130.81 116.84 0)
 			(effects
 				(font
@@
 			)
 		)
-		(property "Datasheet" "http://www.osram-os.com/Graphics/XPic0/00203825_0.pdf"
+		(property "Datasheet" "~"
 			(at 130.81 116.84 0)
 			(effects
@@
 			)
 		)
-		(property "Description" "850nm High Power Infrared Emitter, Side-Emitter package"
-			(at 130.81 115.57 0)
+		(property "Description" "WHITE Rectangular LED, diffused"
+			(at 130.81 116.84 0)
+			(effects
+				(font
+					(size 1.27 1.27)
+				)
+				(hide yes)
+			)
+		)
+		(property "Sim.Pins" "1=K 2=A"
+			(at 130.81 116.84 0)
 			(effects
 				(font
@@
 	)
 	(symbol
-		(lib_id "LED:IRL81A")
-		(at 152.4 115.57 90)
+		(lib_id "Device:LED")
+		(at 152.4 116.84 90)
 		(unit 1)
 		(exclude_from_sim no)
@@
 		(fields_autoplaced yes)
 		(property "Reference" "D3"
-			(at 154.94 115.4429 90)
+			(at 156.21 117.1574 90)
 			(effects
 				(font
@@
 		)
 		(property "Value" "Yellow"
-			(at 154.94 117.9829 90)
+			(at 156.21 119.6974 90)
 			(effects
 				(font
@@
 			)
 		)
-		(property "Footprint" "LED_THT:LED_SideEmitter_Rectangular_W4.5mm_H1.6mm"
-			(at 147.955 115.57 0)
+		(property "Footprint" "LED_THT:LED_Rectangular_W5.0mm_H2.0mm"
+			(at 152.4 116.84 0)
+			(effects
+				(font
+					(size 1.27 1.27)
+				)
+				(hide yes)
+			)
+		)
+		(property "Datasheet" "~"
+			(at 152.4 116.84 0)
 			(effects
 				(font
@@
 			)
 		)
-		(property "Datasheet" "http://www.osram-os.com/Graphics/XPic0/00203825_0.pdf"
+		(property "Description" "YELLOW Rectangular LED, diffused"
 			(at 152.4 116.84 0)
 			(effects
@@
 			)
 		)
-		(property "Description" "850nm High Power Infrared Emitter, Side-Emitter package"
-			(at 152.4 115.57 0)
+		(property "Sim.Pins" "1=K 2=A"
+			(at 152.4 116.84 0)
 			(effects
 				(font
@@
 	)
 	(symbol
-		(lib_id "LED:IRL81A")
-		(at 173.99 115.57 90)
+		(lib_id "Device:LED")
+		(at 173.99 116.84 90)
 		(unit 1)
 		(exclude_from_sim no)
@@
 		(fields_autoplaced yes)
 		(property "Reference" "D6"
-			(at 176.53 115.4429 90)
+			(at 177.8 117.1574 90)
 			(effects
 				(font
@@
 		)
 		(property "Value" "Red"
-			(at 176.53 117.9829 90)
+			(at 177.8 119.6974 90)
 			(effects
 				(font
@@
 			)
 		)
-		(property "Footprint" "LED_THT:LED_SideEmitter_Rectangular_W4.5mm_H1.6mm"
-			(at 169.545 115.57 0)
+		(property "Footprint" "LED_THT:LED_Rectangular_W5.0mm_H2.0mm"
+			(at 173.99 116.84 0)
 			(effects
 				(font
@@
 			)
 		)
-		(property "Datasheet" "http://www.osram-os.com/Graphics/XPic0/00203825_0.pdf"
+		(property "Datasheet" "~"
 			(at 173.99 116.84 0)
 			(effects
@@
 			)
 		)
-		(property "Description" "850nm High Power Infrared Emitter, Side-Emitter package"
-			(at 173.99 115.57 0)
+		(property "Description" "RED Rectangular LED, diffused"
+			(at 173.99 116.84 0)
+			(effects
+				(font
+					(size 1.27 1.27)
+				)
+				(hide yes)
+			)
+		)
+		(property "Sim.Pins" "1=K 2=A"
+			(at 173.99 116.84 0)
 			(effects
 				(font
