File: Oblique Palette 0.5.x PCB Files/Oblique Palette 0.5.1 PCB Input/Oblique Palette 0.5.1 PCB Input.kicad_sch (KiCad schematic)
At the start: 0 parts

Commit message: Associated Input and Output tiles relatively rather than absolutely, which got them lost in the sauce.
Parts:
- added C9: 1n, Capacitor_SMD:C_0805_2012Metric, symbol Device:C
- added D2: White, LED_THT:LED_Rectangular_W5.0mm_H2.0mm, symbol Device:LED
- added D3: Yellow, LED_THT:LED_Rectangular_W5.0mm_H2.0mm, symbol Device:LED
- added D4, D5: 1N4148, Diode_SMD:D_SOD-123, symbol Device:D
- added D6: Red, LED_THT:LED_Rectangular_W5.0mm_H2.0mm, symbol Device:LED
- added J16: Conn_01x03_Female_Pin, Connector_PinSocket_2.54mm:PinSocket_1x03_P2.54mm_Vertical, symbol Connector:Conn_01x03_Pin
- added J17: AudioJack2_SwitchT, Connector_Audio:Jack_3.5mm_QingPu_WQP-PJ398SM_Vertical_CircularHoles, symbol Connector_Audio:AudioJack2_SwitchT
- added R160: 200K, Resistor_SMD:R_0805_2012Metric, symbol Device:R
- added R3: 1K, Resistor_SMD:R_0805_2012Metric, symbol Device:R
- added R4: 300k, Resistor_SMD:R_0805_2012Metric, symbol Device:R
- added R5, R7: 127R, Resistor_SMD:R_0805_2012Metric, symbol Device:R
- added R6: 110K, Resistor_SMD:R_0805_2012Metric, symbol Device:R
- added R68: 100K, Resistor_SMD:R_0805_2012Metric, symbol Device:R
- added R8: 150K, Resistor_SMD:R_0805_2012Metric, symbol Device:R
- added RV1: R_Potentiometer_MountingPin, Potentiometer_THT:Potentiometer_Alps_RK09K_Single_Vertical, symbol Device:R_Potentiometer_MountingPin
- added U3: MCP6004, Package_SO:SOIC-14_3.9x8.7mm_P1.27mm, symbol Amplifier_Operational:MCP6004
Connections:
- new net: J16.1 (Pin_1), R68.1, RV1.2, U3.10 (+), U3.12 (+)
- new net: R160.1, R68.2, U3.3 (+), U3.5 (+)
- new net: C9.1, D4.2 (A), D5.1 (K), J17.T, RV1.3
- new net: D6.1 (K), R7.1
- new net: D3.2 (A), U3.8
- new net: R4.2, R6.1, U3.9 (-)
- new net: D2.1 (K), R3.1, U3.6 (-)
- new net: D2.2 (A), U3.7
- new net: R6.2, R8.1, U3.13 (-)
- new net: D6.2 (A), U3.14
- new net: D3.1 (K), R5.1
- new net +3.3V: U3.4 (V+)
- new net ANALOG_CHANNEL: U3.1, U3.2 (-)
- new net GNDREF: C9.2, D5.2 (A), J16.3 (Pin_3), J17.S, R160.2, R3.2, R4.1, R5.2, R7.2, RV1.1, U3.11 (V-)
- new net VCC: D4.1 (K), J16.2 (Pin_2), J17.TN, R8.2
- no-connect marks 0 -> 1
