File: Oblique Palette 0.5.x PCB Files/Oblique Palette 0.5.1 PCB Output/Oblique Palette 0.5.1 PCB Output.kicad_sch (KiCad schematic)
At the start: 0 parts

Commit message: Associated Input and Output tiles relatively rather than absolutely, which got them lost in the sauce.
Parts:
- added D50: White, LED_THT:LED_Rectangular_W5.0mm_H2.0mm, symbol Device:LED
- added D51: Yellow, LED_THT:LED_Rectangular_W5.0mm_H2.0mm, symbol Device:LED
- added D52: Red, LED_THT:LED_Rectangular_W5.0mm_H2.0mm, symbol Device:LED
- added J40: Conn_01x03_Female_Pin, Connector_PinSocket_2.54mm:PinSocket_1x03_P2.54mm_Vertical, symbol Connector:Conn_01x03_Pin
- added J42: AudioJack2_SwitchT, Connector_Audio:Jack_3.5mm_QingPu_WQP-PJ398SM_Vertical_CircularHoles, symbol Connector_Audio:AudioJack2_SwitchT
- added R112: 200k, Resistor_SMD:R_0805_2012Metric, symbol Device:R
- added R153: 100k, Resistor_SMD:R_0805_2012Metric, symbol Device:R
- added R25: 100R, Resistor_SMD:R_0805_2012Metric, symbol Device:R
- added R69: 300k, Resistor_SMD:R_0805_2012Metric, symbol Device:R
- added R70: 110k, Resistor_SMD:R_0805_2012Metric, symbol Device:R
- added R71: 150k, Resistor_SMD:R_0805_2012Metric, symbol Device:R
- added R73: 1K, Resistor_SMD:R_0805_2012Metric, symbol Device:R
- added R74, R75: 127R, Resistor_SMD:R_0805_2012Metric, symbol Device:R
- added U11: MCP4725xxx-xCH, Package_TO_SOT_SMD:SOT-23-6, symbol Analog_DAC:MCP4725xxx-xCH
- added U12: MCP6004, Package_SO:SOIC-14_3.9x8.7mm_P1.27mm, symbol Amplifier_Operational:MCP6004
Connections:
- new net: R153.2, U11.1 (VOUT)
- new net: J40.1 (Pin_1), J42.T, R25.1
- new net: R25.2, U12.1, U12.2 (-)
- new net: R112.2, R153.1, U12.10 (+), U12.12 (+), U12.3 (+), U12.5 (+)
- new net: D50.1 (K), R73.1, U12.6 (-)
- new net: D50.2 (A), U12.7
- new net: R70.1, R71.2, U12.13 (-)
- new net: R69.1, R70.2, U12.9 (-)
- new net: D51.2 (A), U12.8
- new net: D51.1 (K), R74.1
- new net: D52.2 (A), U12.14
- new net: D52.1 (K), R75.1
- new net +3.3V: R71.1
- new net DAC_ADDR: U11.6 (A0)
- new net GNDREF: J40.3 (Pin_3), J42.S, R112.1, R69.2, R73.2, R74.2, R75.2, U11.2 (VSS), U12.11 (V-)
- new net SERIAL_CLOCK_: U11.5 (SCL)
- new net SERIAL_DATA_: U11.4 (SDA)
- new net VCC: J40.2 (Pin_2), U11.3 (VDD), U12.4 (V+)
- no-connect marks 0 -> 1
